File: hardware/03_afe_ch2.kicad_sch (KiCad schematic)
At the start: 0 parts

Commit message: AFE channel 2: copy of channel 1
Parts:
- added C10, C11: 5-60pF, symbol Device:C_Variable
- added C12: 100nF, Package_SO:SOIC-8_3.9x4.9mm_P1.27mm, symbol Device:C
- added C13, C14: 2.2nF C0G, Package_SO:SOIC-8_3.9x4.9mm_P1.27mm, symbol Device:C
- added D2: BAV99, Package_TO_SOT_SMD:SOT-23, symbol Diode:BAV99
- added J3: BNC_CH2, symbol Connector:Conn_Coaxial
- added R7: 750k, symbol Device:R
- added R8: 250k, symbol Device:R
- added R9: 150R, symbol Device:R
- added U4: MCP6292, Package_TO_SOT_SMD:SOT-353_SC-70-5, symbol Amplifier_Operational:Opamp_Dual
Connections:
- new net: U4.6 (-), U4.7
- new net: R9.1, U4.1, U4.2 (-)
- new net: C10.1, J3.1 (In), R7.1
- new net: C10.2, C11.1, D2.3 (K), R7.2, R8.1, U4.3 (+)
- new net +3V3_A: C12.1, D2.2 (A), U4.8 (V+)
- new net CH2_ANALOG: C13.1, C14.1, R9.2
- new net GND: C12.2, C13.2, C14.2, D2.1 (K), J3.2 (Ext), U4.4 (V-), U4.5 (+)
- new net VREF_2V2: C11.2, R8.2
Other:
- note added: "Anti-alias + Riso + charge bucket. fc = 241kHz. R9 <= 200 ohm per ADS7883 SLAS594 p.11. C0G REQUIRED: X7R drifts with temp and DC bias, which would move the corner frequency."
- note added: "Buffer: divider output impedance = 750k||250k = 188k. ADS7883 needs source impedance < 200 ohm (SLAS594 p.11, "Driving the VIN and VDD Pins"). Buffer makes it a few ohms. MCP6292 rail-to-rail I/O, GBW 10MHz (DS20001812)."
- note added: "Compensation: adjust C10 so R7*C10 = R8*C11 Tune with 1kHz square wave: flat top = correct, sagging = undercomp, overshoot = overcomp."
- note added: "Protection: R7 (750k) limits fault current. 100V fault -> 133uA. BAV99 rated well above this. D2 limits voltage to rail +/- one diode drop. ADS7883 abs max on VIN: -0.3V to VDD+0.3V (SLAS594 p.2)"
- note added: "R7/R8 values are NOMINAL. Measure the actual pair on the DMM and store the measured ratio as a calibration constant in firmware (oscil_cal.h). Ratio sets gain; sum sets input Z. Absolute value does not matter, matching does."
- note added: "Single-ended, NOT isolated. Shell = system GND = USB GND = mains earth. Max +/-5V direct, +/-50V with 10x probe. NEVER connect to mains."
- note added: "space reserved for ADC driver stage if settling is marginal at 2MSa/s"

Commit message: Add final Rev A schematic PDF and edited footprints
Parts:
- C10, C11: footprint (none) -> Capacitor_SMD:C_Trimmer_Murata_TZB4-A
- C12, C13, C14: footprint Package_SO:SOIC-8_3.9x4.9mm_P1.27mm -> Capacitor_THT:C_Disc_D5.0mm_W2.5mm_P5.00mm
- J3: footprint (none) -> Connector_Coaxial:BNC_PanelMountable_Vertical
- R7, R8, R9: footprint (none) -> Resistor_THT:R_Axial_DIN0207_L6.3mm_D2.5mm_P10.16mm_Horizontal
- U4: footprint Package_TO_SOT_SMD:SOT-353_SC-70-5 -> Package_DIP:DIP-8_W7.62mm
Changed lines of the file:
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@@
 	(title_block
 		(title "Oscil")
-		(date "2026-09-18")
-		(rev "0.1")
+		(date "2026-09-21")
+		(rev "A")
 		(comment 1 "Two-channel Digital Oscilloscope and Function Generator")
 		(comment 2 "ESP32-S3 / ESP-IDF / FreeRTOS")
@@
 			)
 		)
-		(property "Footprint" "Package_TO_SOT_SMD:SOT-353_SC-70-5"
+		(property "Footprint" "Package_DIP:DIP-8_W7.62mm"
 			(at 168.91 81.28 0)
 			(hide yes)
@@
 			)
 		)
-		(property "Footprint" "Package_SO:SOIC-8_3.9x4.9mm_P1.27mm"
+		(property "Footprint" "Capacitor_THT:C_Disc_D5.0mm_W2.5mm_P5.00mm"
 			(at 141.9352 76.2 0)
 			(hide yes)
@@
 			)
 		)
-		(property "Footprint" ""
+		(property "Footprint" "Resistor_THT:R_Axial_DIN0207_L6.3mm_D2.5mm_P10.16mm_Horizontal"
 			(at 153.67 48.768 90)
 			(hide yes)
@@
 			)
 		)
-		(property "Footprint" ""
+		(property "Footprint" "Capacitor_SMD:C_Trimmer_Murata_TZB4-A"
 			(at 88.9 44.45 0)
 			(hide yes)
@@
 			)
 		)
-		(property "Footprint" ""
+		(property "Footprint" "Connector_Coaxial:BNC_PanelMountable_Vertical"
 			(at 49.53 40.64 0)
 			(hide yes)
@@
 			)
 		)
-		(property "Footprint" "Package_TO_SOT_SMD:SOT-353_SC-70-5"
+		(property "Footprint" "Package_DIP:DIP-8_W7.62mm"
 			(at 135.89 46.99 0)
 			(hide yes)
@@
 			)
 		)
-		(property "Footprint" "Package_SO:SOIC-8_3.9x4.9mm_P1.27mm"
+		(property "Footprint" "Capacitor_THT:C_Disc_D5.0mm_W2.5mm_P5.00mm"
 			(at 169.8752 54.61 0)
 			(hide yes)
@@
 			)
 		)
-		(property "Footprint" "Package_TO_SOT_SMD:SOT-353_SC-70-5"
+		(property "Footprint" "Package_DIP:DIP-8_W7.62mm"
 			(at 134.62 71.12 0)
 			(hide yes)
@@
 			)
 		)
-		(property "Footprint" "Package_SO:SOIC-8_3.9x4.9mm_P1.27mm"
+		(property "Footprint" "Capacitor_THT:C_Disc_D5.0mm_W2.5mm_P5.00mm"
 			(at 162.2552 54.61 0)
 			(hide yes)
@@
 			)
 		)
-		(property "Footprint" ""
+		(property "Footprint" "Resistor_THT:R_Axial_DIN0207_L6.3mm_D2.5mm_P10.16mm_Horizontal"
 			(at 71.882 45.72 90)
 			(hide yes)
@@
 			)
 		)
-		(property "Footprint" ""
+		(property "Footprint" "Capacitor_SMD:C_Trimmer_Murata_TZB4-A"
 			(at 88.9 60.96 0)
 			(hide yes)
@@
 			)
 		)
-		(property "Footprint" ""
+		(property "Footprint" "Resistor_THT:R_Axial_DIN0207_L6.3mm_D2.5mm_P10.16mm_Horizontal"
 			(at 71.882 60.96 90)
 			(hide yes)
